File: kicadpractice/kicadpractice.kicad_pcb (KiCad board)
At the start: 2 copper layers, 9 parts, among them SW1 SW_SPST, SW2 SW_SPST, SW3 SW_SPST

Commit message: 2026-06-15(2)
Parts:
- added H1: MountingHole_Pad, MountingHole:MountingHole_3.2mm_M3_ISO14580_Pad, F.Cu at (5.25, 5.25)
- added H2: MountingHole_Pad, MountingHole:MountingHole_3.2mm_M3_ISO14580_Pad, F.Cu at (5.25, 44.8)
- added H3: MountingHole_Pad, MountingHole:MountingHole_3.2mm_M3_ISO14580_Pad, F.Cu at (54.8, 5.25)
- added H4: MountingHole_Pad, MountingHole:MountingHole_3.2mm_M3_ISO14580_Pad, F.Cu at (54.8, 44.5)
- added J1: Jack-DC, Connector_BarrelJack:BarrelJack_GCT_DCJ200-10-A_Horizontal, F.Cu at (14.8, 25.5)
- moved SW2 135.1 mm to (21.0, 23.0)
- moved R1 134.4 mm to (35.2, 9.00)
- moved R2 133.8 mm to (37.2, 23.0)
- moved SW3 131.8 mm to (21.0, 37.8)
- moved SW1 128.7 mm to (21.0, 8.50)
- moved R3 127.5 mm to (37.2, 39.0)
- moved D1 125.8 mm to (50.0, 10.5), turned to 180 degrees
- moved D2 121.4 mm to (50.0, 25.0), turned to 180 degrees
- moved D3 116.7 mm to (50.0, 40.2), turned to 180 degrees
Routing:
- added copper zone on F.Cu, net VCC
Other:
- board outline added: 60 x 50 mm

Commit message: 2026-06-16
Parts:
- added G***: LOGO, LOGO, F.Cu at (5.25, 36.5)
- moved D3 2.08 mm to (47.9, 40.2)
Routing:
- net VCC: track 0.00 -> 64.0 mm
- net Net-(SW2-B): track 0.00 -> 18.7 mm, vias 0 -> 1
- net Net-(SW3-B): track 0.00 -> 18.1 mm
- net Net-(SW1-B): track 0.00 -> 16.9 mm
- net Net-(D2-A): track 0.00 -> 10.0 mm
- net Net-(D1-A): track 0.00 -> 7.79 mm
- net Net-(D3-A): track 0.00 -> 7.74 mm
- net GND: vias 0 -> 31
- added copper zone on B.Cu, net GND
- added copper zone on F.Cu, net GND
Other:
- board text added: "led test"

Commit message: 2026-06-24
Parts:
- moved H2 63.7 mm to (55.0, 5.00)
- moved H4 49.8 mm to (5.00, 45.0)
- moved H3 39.8 mm to (55.0, 45.0)
- moved G*** 7.92 mm to (12.5, 39.7)
- moved SW3 3.75 mm to (24.0, 35.5)
- moved R2 3.40 mm to (40.0, 25.0)
- moved R3 3.40 mm to (40.5, 38.0)
- moved SW2 3.35 mm to (24.0, 21.5)
- moved D3 3.22 mm to (50.2, 38.0)
- moved SW1 3.04 mm to (24.0, 8.00)
- moved R1 2.46 mm to (37.5, 10.0)
- moved J1 0.90 mm to (15.5, 25.0)
- moved D1 0.55 mm to (50.2, 10.0)
- moved H1 0.35 mm to (5.00, 5.00)
- moved D2 0.23 mm to (50.2, 25.0)
Routing:
- net VCC: track 64.0 -> 0.00 mm
- net Net-(D2-A): track 10.0 -> 6.69 mm
- net Net-(SW2-B): track 18.7 -> 15.4 mm, vias 1 -> 0
- net Net-(D1-A): track 7.79 -> 5.15 mm
- net Net-(SW1-B): track 16.9 -> 14.5 mm
- net Net-(SW3-B): track 18.1 -> 16.4 mm
- net Net-(D3-A): track 7.74 -> 6.27 mm
- net GND: vias 31 -> 57
- removed copper zone on B.Cu, net GND
Other:
- board text added: "Minu"
- board text removed: "led test"

Commit message: 2026-06-25
Parts:
- added J2: 1612898-1, kicadpracticefootprint:TE_1612898-1, F.Cu at (71.1, 42.5)

Commit message: 2026-06-27
Parts:
- added D10: LED, minuchok's_footprints:LED_D5.0mm_centered, F.Cu at (135.4, -44.6)
- added D11: LED, minuchok's_footprints:LED_D5.0mm_centered, F.Cu at (119.1, -33.8)
- added D12: LED, minuchok's_footprints:LED_D5.0mm_centered, F.Cu at (100.0, -30.0)
- added D13: LED, minuchok's_footprints:LED_D5.0mm_centered, F.Cu at (80.9, -33.8)
- added D14: LED, minuchok's_footprints:LED_D5.0mm_centered, F.Cu at (64.6, -44.6)
- added D15: LED, minuchok's_footprints:LED_D5.0mm_centered, F.Cu at (53.8, -60.9)
- added D16: LED, minuchok's_footprints:LED_D5.0mm_centered, F.Cu at (50.0, -80.0)
- added D17: LED, minuchok's_footprints:LED_D5.0mm_centered, F.Cu at (53.8, -99.1)
- added D18: LED, minuchok's_footprints:LED_D5.0mm_centered, F.Cu at (64.6, -115.4)
- added D19: LED, minuchok's_footprints:LED_D5.0mm_centered, F.Cu at (80.9, -126.2)
- added D4: LED, LED_THT:LED_D5.0mm, F.Cu at (100.0, -130.0)
- added D5: LED, minuchok's_footprints:LED_D5.0mm_centered, F.Cu at (119.1, -126.2)
- added D6: LED, minuchok's_footprints:LED_D5.0mm_centered, F.Cu at (135.4, -115.4)
- added D7: LED, minuchok's_footprints:LED_D5.0mm_centered, F.Cu at (146.2, -99.1)
- added D8: LED, minuchok's_footprints:LED_D5.0mm_centered, F.Cu at (150.0, -80.0)
- added D9: LED, minuchok's_footprints:LED_D5.0mm_centered, F.Cu at (146.2, -60.9)
Other:
- board size 60 x 50 mm -> 160 x 200 mm
- board text added: "1"
- board text added: "10"
- board text added: "11"
- board text added: "12"
- board text added: "13"
- board text added: "14"
- board text added: "15"
- board text added: "16"
- board text added: "2"
- board text added: "3"
- board text added: "4"
- board text added: "5"
- board text added: "6"
- board text added: "7"
- board text added: "8"
- board text added: "9"
