File: kicadpractice/kicadpractice.kicad_sch (KiCad schematic)
At the start: 0 parts

Commit message: 2026-06-14
Parts:
- added D1, D2, D3: LED, LED_THT:LED_D5.0mm, symbol Device:LED
- added J1: Jack-DC, symbol Connector:Jack-DC
- added R1: 330R(1/8W), Resistor_THT:R_Axial_DIN0204_L3.6mm_D1.6mm_P5.08mm_Horizontal, symbol Device:R_US
- added R2: 330R(2012), Resistor_SMD:R_0805_2012Metric_Pad1.20x1.40mm_HandSolder, symbol Device:R_US
- added R3: 330R(1608), Resistor_SMD:R_0603_1608Metric_Pad0.98x0.95mm_HandSolder, symbol Device:R_US
- added SW1, SW2, SW3: SW_SPST, Button_Switch_THT:SW_PUSH_6mm_H5mm, symbol Switch:SW_SPST
Connections:
- new net: R3.1, SW3.2 (B)
- new net: D3.2 (A), R3.2
- new net: R2.1, SW2.2 (B)
- new net: D1.2 (A), R1.2
- new net: D2.2 (A), R2.2
- new net: R1.1, SW1.2 (B)
- new net GND: D1.1 (K), D2.1 (K), D3.1 (K), J1.2
- new net VCC: J1.1, SW1.1 (A), SW2.1 (A), SW3.1 (A)

Commit message: 2026-06-15(2)
Parts:
- added H1, H2, H3, H4: MountingHole_Pad, MountingHole:MountingHole_3.2mm_M3_ISO14580_Pad, symbol Mechanical:MountingHole_Pad
- J1: footprint (none) -> Connector_BarrelJack:BarrelJack_GCT_DCJ200-10-A_Horizontal
Other:
- moved on the sheet: D3, R3, SW3

Commit message: 2026-06-25
Parts:
- added J2: 1612898-1, kicadpracticefootprint:TE_1612898-1, symbol New_Library:1612898-1
Changed lines of the file:
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@@
+	)
+	(symbol
+		(lib_id "New_Library:1612898-1")
+		(at 128.27 90.17 0)
+		(unit 1)
+		(body_style 1)
+		(exclude_from_sim no)
+		(in_bom yes)
+		(on_board yes)
+		(in_pos_files yes)
+		(dnp no)
+		(fields_autoplaced yes)
+		(property "Reference" "J2"
+			(at 120.65 82.55 0)
+			(show_name no)
+			(do_not_autoplace no)
+			(effects
+				(font
+					(size 1.27 1.27)
+				)
+			)
+		)
+		(property "Value" "1612898-1"
+			(at 120.65 85.09 0)
+			(show_name no)
+			(do_not_autoplace no)
+			(effects
+				(font
+					(size 1.27 1.27)
+				)
+			)
+		)
+		(property "Footprint" "kicadpracticefootprint:TE_1612898-1"
+			(at 128.27 90.17 0)
+			(hide yes)
+			(show_name no)
+			(do_not_autoplace no)
+			(effects
+				(font
+					(size 1.27 1.27)
+				)
+				(justify bottom)
+			)
+		)
+		(property "Datasheet" ""
+			(at 128.27 90.17 0)
+			(hide yes)
+			(show_name no)
+			(do_not_autoplace no)
+			(effects
+				(font
+					(size 1.27 1.27)
+				)
+			)
+		)
+		(property "Description" ""
+			(at 128.27 90.17 0)
+			(hide yes)
+			(show_name no)
+			(do_not_autoplace no)
+			(effects
+				(font
+					(size 1.27 1.27)
+				)
+			)
+		)
+		(property "MAXIMUM_PACKAGE_HEIGHT" "5.4mm"
+			(at 128.27 90.17 0)
+			(hide yes)
+			(show_name no)
+			(do_not_autoplace no)
+			(effects
+				(font
+					(size 1.27 1.27)
+				)
+				(justify bottom)
+			)
+		)
+		(property "CREATOR" "ASHISH"
+			(at 128.27 90.17 0)
+			(hide yes)
+			(show_name no)
+			(do_not_autoplace no)
+			(effects
+				(font
+					(size 1.27 1.27)
+				)
+				(justify bottom)
+			)
+		)
+		(property "STANDARD" "Manufacturer Recommendations"
+			(at 128.27 90.17 0)
+			(hide yes)
+			(show_name no)
+			(do_not_autoplace no)
+			(effects
+				(font
+					(size 1.27 1.27)
+				)
+				(justify bottom)
+			)
+		)
+		(property "PARTREV" "O"
+			(at 128.27 90.17 0)
+			(hide yes)
+			(show_name no)
+			(do_not_autoplace no)
+			(effects
+				(font
+					(size 1.27 1.27)
+				)
+				(justify bottom)
+			)
+		)
+		(property "VERIFIER" ""
+			(at 128.27 90.17 0)
+			(hide yes)
+			(show_name no)
+			(do_not_autoplace no)
+			(effects
+				(font
+					(size 1.27 1.27)
+				)
+				(justify bottom)
+			)
+		)
+		(property "CAD_BUILD" "TE OEM"
+			(at 128.27 90.17 0)
+			(hide yes)
+			(show_name no)
+			(do_not_autoplace no)
+			(effects
+				(font
+					(size 1.27 1.27)
+				)
+				(justify bottom)
+			)
+		)
+		(property "MANUFACTURER" "TE Connectivity"
+			(at 128.27 90.17 0)
+			(hide yes)
+			(show_name no)
+			(do_not_autoplace no)
+			(effects
+				(font
+					(size 1.27 1.27)
+				)
+				(justify bottom)
+			)
+		)
+		(pin "1_2"
+		)
+		(pin "2_1"
+		)
+		(pin "3_1"
+		)
+		(pin "2_3"
+		)
+		(pin "3_2"
+		)
+		(pin "3_3"
+		)
+		(pin "1_1"
+		)
+		(pin "1_3"
+		)
+		(pin "2_2"
+		)
+		(instances
+			(project "kicadpractice"
+				(path "/ac7dd70a-53cb-4ff2-b438-62369eca99c9"
+					(reference "J2")
+					(unit 1)
+				)
+			)
+		)
 	)
 	(symbol

Commit message: 2026-06-27
Parts:
- added D10, D11, D12, D13, D14, D15, D16, D17, D18, D19, D4, D5, D6, D7, D8, D9: LED, LED_THT:LED_D5.0mm, symbol Device:LED
