File: kicadpractice/kicadembeded/kicadembeded.kicad_sch (KiCad schematic)
At the start: 0 parts

Commit message: 2026-06-28
Parts:
- added D1: LED, LED_THT:LED_D5.0mm, symbol Device:LED
- added J1: Conn_ARM_JTAG_SWD_20, symbol Connector:Conn_ARM_JTAG_SWD_20
- added R1: 17K, symbol Device:R_US
- added R2: 33K, symbol Device:R_US
- added R3: 130, symbol Device:R_US
Connections:
- new net: R1.1, R2.2, R3.2
- new net: D1.2 (A), R3.1
- new net GND: D1.1 (K), J1.10 (GND), J1.12 (GND), J1.14 (GND), J1.16 (GND), J1.18 (GND), J1.20 (GND), J1.4 (GND), J1.6 (GND), J1.8 (GND), R2.1
- new net VCC: J1.2 (VCC/NC), R1.2
